File: hardware/schemTSC.sch (EAGLE design)
At the start: 105 parts, among them IC1 BQ25180YBGR, IC2 DRV2605YZFR, IC3 BMA421, IC9 RT6160AWSC, J1 503480-2400, J2 TC2030-IDC, J4 KH-TYPE-C-16P, Q3 SI1308EDL-T1-GE3, U1 NRF52840_QF, U3 MAX17048G+T10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

Commit message: Add files via upload
Connections:
- removed net N$33: C31.2, R8.1
- removed net N$36: C29.2, R7.1
- removed net OUT: IC2.OUT-
- net OUT-: now also IC2.OUT-
- net P0.14/1.5D: now also C31.2, R8.1
- net P1.02/1.6C: now also C29.2, R7.1
Changed lines of the file:
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@@
 <instance part="ANT1" gate="G$1" x="251.46" y="607.06" smashed="yes">
 <attribute name="NAME" x="252.73" y="617.22" size="1.778" layer="95" align="center-left"/>
-<attribute name="VALUE" x="232.41" y="614.68" size="1.778" layer="96" align="center-left"/>
+<attribute name="VALUE" x="247.65" y="612.14" size="1.778" layer="96" align="center-left"/>
 </instance>
 <instance part="C11" gate="C$1" x="175.26" y="640.08" smashed="yes">
@@
 <pinref part="SW_DN" gate="A" pin="1"/>
 <wire x1="215.9" y1="259.08" x2="215.9" y2="251.46" width="0.1524" layer="91"/>
-<junction x="220.98" y="251.46"/>
 <wire x1="220.98" y1="251.46" x2="220.98" y2="248.92" width="0.1524" layer="91"/>
 <pinref part="SUPPLY53" gate="G$1" pin="GND"/>
+<junction x="220.98" y="251.46"/>
 </segment>
 <segment>
@@
 </segment>
 </net>
-<net name="OUT" class="0">
-<segment>
-<pinref part="IC2" gate="G$1" pin="OUT-"/>
-<wire x1="223.52" y1="360.68" x2="226.06" y2="360.68" width="0.1524" layer="91"/>
-<label x="226.06" y="360.68" size="1.778" layer="95" xref="yes"/>
-</segment>
-</net>
 <net name="SDA/1.4C" class="0">
 <segment>
@@
 <wire x1="246.38" y1="393.7" x2="243.84" y2="393.7" width="0.1524" layer="91"/>
 <label x="243.84" y="393.7" size="1.778" layer="95" rot="R180" xref="yes"/>
+</segment>
+<segment>
+<pinref part="IC2" gate="G$1" pin="OUT-"/>
+<wire x1="223.52" y1="360.68" x2="226.06" y2="360.68" width="0.1524" layer="91"/>
+<label x="226.06" y="360.68" size="1.778" layer="95" xref="yes"/>
 </segment>
 </net>
@@
 </segment>
 </net>
-<net name="N$33" class="0">
-<segment>
-<pinref part="R8" gate="G$1" pin="1"/>
-<wire x1="203.2" y1="281.94" x2="203.2" y2="271.78" width="0.1524" layer="91"/>
-<pinref part="C31" gate="G$1" pin="2"/>
-</segment>
-</net>
 <net name="P0.14/1.5D" class="0">
 <segment>
 <pinref part="SW_ENT" gate="A" pin="2"/>
 <wire x1="193.04" y1="274.32" x2="193.04" y2="276.86" width="0.1524" layer="91"/>
-<wire x1="193.04" y1="276.86" x2="205.74" y2="276.86" width="0.1524" layer="91"/>
+<wire x1="193.04" y1="276.86" x2="203.2" y2="276.86" width="0.1524" layer="91"/>
 <label x="205.74" y="276.86" size="1.016" layer="95" xref="yes"/>
-</segment>
-</net>
-<net name="N$36" class="0">
-<segment>
-<wire x1="226.06" y1="281.94" x2="226.06" y2="271.78" width="0.1524" layer="91"/>
-<pinref part="R7" gate="G$1" pin="1"/>
-<pinref part="C29" gate="G$1" pin="2"/>
+<pinref part="R8" gate="G$1" pin="1"/>
+<pinref part="C31" gate="G$1" pin="2"/>
+<wire x1="203.2" y1="271.78" x2="203.2" y2="276.86" width="0.1524" layer="91"/>
+<wire x1="203.2" y1="276.86" x2="203.2" y2="281.94" width="0.1524" layer="91"/>
+<junction x="203.2" y="276.86"/>
+<wire x1="203.2" y1="276.86" x2="205.74" y2="276.86" width="0.1524" layer="91"/>
 </segment>
 </net>
 <net name="P1.02/1.6C" class="0">
 <segment>
-<wire x1="215.9" y1="274.32" x2="228.6" y2="274.32" width="0.1524" layer="91"/>
+<wire x1="215.9" y1="274.32" x2="226.06" y2="274.32" width="0.1524" layer="91"/>
 <pinref part="SW_DN" gate="A" pin="2"/>
 <label x="228.6" y="274.32" size="1.016" layer="95" xref="yes"/>
-</segment>
-</net>
+<pinref part="C29" gate="G$1" pin="2"/>
+<wire x1="226.06" y1="274.32" x2="228.6" y2="274.32" width="0.1524" layer="91"/>
+<wire x1="226.06" y1="271.78" x2="226.06" y2="274.32" width="0.1524" layer="91"/>
+<junction x="226.06" y="274.32"/>
+<wire x1="226.06" y1="274.32" x2="226.06" y2="281.94" width="0.1524" layer="91"/>
+<pinref part="R7" gate="G$1" pin="1"/>
+</segment>
+</net>

Commit message: Loaded all finished files
Connections:
- removed net N$21: J1.MP2
- removed net N$26: EPD_C2.1
- removed net N$27: EPD_C1.1
- net GND: now also C27.1, EPD_C1.1, EPD_C2.1, J1.MP2
Other:
- note added: "drawn by Pascu Eric"
- moved on the sheet: EPD_C12
