File: hardware/schemaPCB.brd (EAGLE design)
At the start: 46 x 35 mm, 105 parts, among them IC1 BQ25180YBGR, IC2 DRV2605YZFR, IC3 BMA421, IC9 RT6160AWSC, J1 503480-2400, J2 TC2030-IDC, J4 KH-TYPE-C-16P, Q3 SI1308EDL-T1-GE3, U1 NRF52840_QF, U3 MAX17048G+T10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

Commit message: Add files via upload
Parts:
- moved C17 97.2 mm to (38.3, 25.4), turned to 90 degrees
- moved C30 93.5 mm to (35.5, 10.5), turned to 180 degrees
- moved C2-EP-DR 91.4 mm to (30.8, 35.3), turned to 270 degrees
- moved C18 90.7 mm to (38.3, 22.9), turned to 90 degrees
- moved TP_VBAT 86.8 mm to (60.7, 9.40)
- moved C29 86.1 mm to (57.1, 10.5), turned to 90 degrees
- moved TP_VREG 84.4 mm to (58.7, 18.0)
- moved C27 81.8 mm to (59.6, 15.8)
- moved TP_SWO 81.3 mm to (48.7, 18.1)
- moved C5 80.3 mm to (41.9, 24.3), turned to 180 degrees
- moved C20 79.8 mm to (42.7, 18.7), turned to 270 degrees
- moved C14 79.5 mm to (41.9, 26.2), turned to 90 degrees
- moved TP_GND 75.9 mm to (62.0, 12.3)
- moved C42 75.2 mm to (40.4, 32.3)
- moved C21 75.0 mm to (45.7, 17.4)
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Connections:
- removed net N$33: C31.2, R8.1
- removed net N$36: C29.2, R7.1
- removed net OUT: IC2.C3
- net OUT-: now also IC2.C3
- net P0.14/1.5D: now also C31.2, R8.1
- net P1.02/1.6C: now also C29.2, R7.1
Routing:
- net GND: track 0.00 -> 419.8 mm, vias 0 -> 20
- net 3V3/2.4A: track 0.00 -> 103.1 mm, vias 0 -> 7
- net SDA/2.4C: track 0.00 -> 72.1 mm, vias 0 -> 5
- net SCL/2.4C: track 0.00 -> 53.5 mm, vias 0 -> 5
- net EPD_3V3: track 0.00 -> 41.3 mm, vias 0 -> 3
- net 3V3/1.7D: track 0.00 -> 38.5 mm, vias 0 -> 2
- net RESET: track 0.00 -> 38.2 mm, vias 0 -> 2
- net SDA/1.4C: track 0.00 -> 33.7 mm, vias 0 -> 2
- net VREG: track 0.00 -> 32.2 mm
- net SCL/1.4C: track 0.00 -> 31.9 mm, vias 0 -> 2
- net PREVGL: track 0.00 -> 29.4 mm
- net SWDCLK: track 0.00 -> 25.4 mm
- net DP: track 0.00 -> 23.4 mm
- net JJ: track 0.00 -> 22.0 mm
- net VBUS/1.5D: track 0.00 -> 21.8 mm, vias 0 -> 2
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
Commit message: Loaded all finished files
Parts:
- moved IC9 0.28 mm to (48.4, 14.7)
- moved C1-EP-DR 0.25 mm to (30.3, 39.8)
Connections:
- removed net N$21: J1.MP2
- removed net N$26: EPD_C2.1
- removed net N$27: EPD_C1.1
- net GND: now also C27.1, EPD_C1.1, EPD_C2.1, J1.MP2
Routing:
- net GND: track 419.8 -> 431.0 mm
- net RESET: track 38.2 -> 35.9 mm
- net SWDCLK: track 25.4 -> 24.4 mm
- net EPD_3V3: track 41.3 -> 40.6 mm
- net N$19: track 3.25 -> 3.76 mm
